Commit message: removed files

File: robot_description/urdf/turtlebot3_burger.urdf.xacro (robot description, xacro)
@@ -113,5 +113,5 @@
   </joint>
   <link name="imu_link"/>
-  <joint name="scan_joint" type="fixed">
+  <!-- <joint name="scan_joint" type="fixed">
     <parent link="base_link"/>
     <child link="base_scan"/>
@@ -139,4 +139,4 @@
                izz="0.001" />
     </inertial>
-  </link>
+  </link> -->
 </robot>
